File: XDS-Analog-to-StudioHub.sch (KiCad schematic (older format))
At the start: 13 parts, among them J1 RJ45_Shielded, J2 DB9_Male

Commit message: Initial Commit
Parts:
- J2: value DB9_Male -> DB9_Female; symbol Connector:DB9_Male_MountingHoles -> Connector:DB9_Female_MountingHoles
Connections:
- net at J2.0 (PAD): no longer JP8.2
- net at J2.2, J2.4, J2.7: no longer JP5.2, JP9.2
- new net: JP5.2, JP9.2
Changed lines of the file:
@@
 $EndComp
 $Comp
-L Connector:DB9_Male_MountingHoles J2
+L Connector:DB9_Female_MountingHoles J2
 U 1 1 60E88828
-P 4800 1550
-F 0 "J2" H 4980 1552 50  0000 L CNN
-F 1 "DB9_Male" H 4980 1461 50  0000 L CNN
-F 2 "Connector_Dsub:DSUB-9_Female_Horizontal_P2.77x2.84mm_EdgePinOffset4.94mm_Housed_MountingHolesOffset7.48mm" H 4800 1550 50  0001 C CNN
-F 3 " ~" H 4800 1550 50  0001 C CNN
-	1    4800 1550
+P 5200 1600
+F 0 "J2" H 5380 1602 50  0000 L CNN
+F 1 "DB9_Female" H 5380 1511 50  0000 L CNN
+F 2 "Connector_Dsub:DSUB-9_Female_Horizontal_P2.77x2.84mm_EdgePinOffset4.94mm_Housed_MountingHolesOffset7.48mm" H 5200 1600 50  0001 C CNN
+F 3 " ~" H 5200 1600 50  0001 C CNN
+	1    5200 1600
 	1    0    0    -1
 $EndComp
@@
 Wire Wire Line
 	3250 1950 3100 1950
-Wire Wire Line
-	3850 1950 4500 1950
 $Comp
 L Device:Jumper JP6
@@
 $EndComp
 Wire Wire Line
-	3850 1800 3850 1850
-Wire Wire Line
-	3850 1850 4500 1850
-Wire Wire Line
 	3250 1800 3150 1800
 Wire Wire Line
@@
 $EndComp
 Wire Wire Line
-	3850 1150 4500 1150
-Wire Wire Line
 	3250 1150 2950 1150
 Wire Wire Line
@@
 $EndComp
 Wire Wire Line
-	3850 1300 3850 1250
-Wire Wire Line
-	3850 1250 4500 1250
-Wire Wire Line
 	3000 1300 3000 1450
 Wire Wire Line
@@
 $EndComp
 Wire Wire Line
-	4800 2150 3850 2150
-Wire Wire Line
 	3250 2150 3050 2150
 $Comp
@@
 NoConn ~ 2700 1350
 NoConn ~ 2700 1250
-Wire Wire Line
-	4500 1750 4500 1650
-Wire Wire Line
-	4500 1650 4350 1650
-Wire Wire Line
-	4350 1650 4350 1550
-Wire Wire Line
-	4350 1350 4500 1350
-Connection ~ 4500 1650
-Connection ~ 4350 1550
-Wire Wire Line
-	4350 1550 4350 1350
 $Comp
 L Device:Jumper JP9
@@
 Wire Wire Line
 	4100 2450 3850 2450
-Connection ~ 4100 1550
 Wire Wire Line
 	4100 1550 3850 1550
@@
 	1    0    0    -1
 $EndComp
-Wire Wire Line
-	4350 1550 4100 1550
-Wire Wire Line
-	4200 1450 4200 1500
-Wire Wire Line
-	4200 1500 4500 1500
-Wire Wire Line
-	4500 1500 4500 1550
-Wire Wire Line
-	4500 1450 4250 1450
-Wire Wire Line
-	4250 1450 4250 1350
-Wire Wire Line
-	4250 1350 4200 1350
 Wire Wire Line
 	4000 1450 3100 1450
@@
 Wire Wire Line
 	2800 1850 2700 1850
+Wire Wire Line
+	3850 1150 4450 1150
+Wire Wire Line
+	4450 1150 4450 2000
+Wire Wire Line
+	4450 2000 4900 2000
+Wire Wire Line
+	3850 1300 4500 1300
+Wire Wire Line
+	4500 1300 4500 1900
+Wire Wire Line
+	4500 1900 4900 1900
+Wire Wire Line
+	3850 1950 4550 1950
+Wire Wire Line
+	4550 1950 4550 1200
+Wire Wire Line
+	4550 1200 4900 1200
+Wire Wire Line
+	3850 1800 4600 1800
+Wire Wire Line
+	4600 1800 4600 1300
+Wire Wire Line
+	4600 1300 4900 1300
+Wire Wire Line
+	4200 1450 4700 1450
+Wire Wire Line
+	4700 1450 4700 1600
+Wire Wire Line
+	4700 1600 4900 1600
+Wire Wire Line
+	4200 1350 4800 1350
+Wire Wire Line
+	4800 1350 4800 1700
+Wire Wire Line
+	4800 1700 4900 1700
+Wire Wire Line
+	4900 1400 4900 1450
+Wire Wire Line
+	4900 1800 4850 1800
+Wire Wire Line
+	4850 1800 4850 1450
+Wire Wire Line
+	4850 1450 4900 1450
+Connection ~ 4900 1450
+Wire Wire Line
+	4900 1450 4900 1500
 $EndSCHEMATC

Commit message: corrected grounding issue
Parts:
- removed JP1: MONO-, Connector_PinHeader_2.54mm:PinHeader_1x02_P2.54mm_Vertical, symbol Device:Jumper_NO_Small
- removed JP2: MONO+, Connector_PinHeader_2.54mm:PinHeader_1x02_P2.54mm_Vertical, symbol Device:Jumper_NO_Small
- JP3, JP4: footprint Connector_PinHeader_2.54mm:PinHeader_1x02_P2.54mm_Vertical -> Connector_PinHeader_2.54mm:PinHeader_1x03_P2.54mm_Vertical; symbol Device:Jumper -> Jumper:Jumper_3_Bridged12
- JP5: value DC-GND -> GND-GND
Connections:
- net at J1.3: now also JP3.2 (C); no longer JP3.1
- net at J1.6: now also JP4.2 (C); no longer JP4.1
- net at J2.0 (PAD): now also JP8.2
- net at J2.1, JP7.2: now also JP3.3 (B)
- net at J2.2, J2.4, J2.7: now also JP5.2, JP9.2
- net at J2.5: now also JP3.1 (A); no longer JP3.2
- net at J2.6, JP6.2: now also JP4.3 (B)
- net at J2.9: now also JP4.1 (A); no longer JP4.2
Changed lines of the file:
@@
 	3150 1850 3050 1850
 $Comp
-L Device:Jumper JP3
+L Jumper:Jumper_3_Bridged12 JP3
 U 1 1 60E96B38
-P 3550 1150
-F 0 "JP3" H 3550 1414 50  0001 C CNN
-F 1 "R+" H 3550 1150 50  0000 C CNN
-F 2 "Connector_PinHeader_2.54mm:PinHeader_1x02_P2.54mm_Vertical" H 3550 1150 50  0001 C CNN
-F 3 "~" H 3550 1150 50  0001 C CNN
-	1    3550 1150
-	1    0    0    -1
-$EndComp
-Wire Wire Line
-	3250 1150 2950 1150
+P 3350 850
+F 0 "JP3" H 3350 1114 50  0001 C CNN
+F 1 "R+" H 3350 950 50  0000 C CNN
+F 2 "Connector_PinHeader_2.54mm:PinHeader_1x03_P2.54mm_Vertical" H 3350 850 50  0001 C CNN
+F 3 "~" H 3350 850 50  0001 C CNN
+	1    3350 850
+	1    0    0    -1
+$EndComp
 Wire Wire Line
 	2950 1150 2950 1750
-Wire Wire Line
-	2950 1750 2850 1750
-$Comp
-L Device:Jumper JP4
+$Comp
+L Jumper:Jumper_3_Bridged12 JP4
 U 1 1 60E98348
-P 3550 1300
-F 0 "JP4" H 3550 1564 50  0001 C CNN
-F 1 "R-" H 3550 1300 50  0000 C CNN
-F 2 "Connector_PinHeader_2.54mm:PinHeader_1x02_P2.54mm_Vertical" H 3550 1300 50  0001 C CNN
-F 3 "~" H 3550 1300 50  0001 C CNN
-	1    3550 1300
+P 4050 850
+F 0 "JP4" H 4050 1114 50  0001 C CNN
+F 1 "R-" H 4050 950 50  0000 C CNN
+F 2 "Connector_PinHeader_2.54mm:PinHeader_1x03_P2.54mm_Vertical" H 4050 850 50  0001 C CNN
+F 3 "~" H 4050 850 50  0001 C CNN
+	1    4050 850
 	1    0    0    -1
 $EndComp
 Wire Wire Line
 	3000 1300 3000 1450
-Wire Wire Line
-	3000 1450 2800 1450
 $Comp
 L Device:Jumper JP8
@@
 P 3550 1550
 F 0 "JP5" H 3550 1814 50  0001 C CNN
-F 1 "DC-GND" H 3550 1450 50  0000 C CNN
+F 1 "GND-GND" H 3550 1450 50  0000 C CNN
 F 2 "Connector_PinHeader_2.54mm:PinHeader_1x02_P2.54mm_Vertical" H 3550 1550 50  0001 C CNN
 F 3 "~" H 3550 1550 50  0001 C CNN
@@
 Connection ~ 3100 1950
 Wire Wire Line
-	3100 1950 2850 1950
-Wire Wire Line
 	4000 1350 3050 1350
 Wire Wire Line
@@
 Connection ~ 3050 1850
 Wire Wire Line
-	3050 1850 2800 1850
-$Comp
-L Device:Jumper_NO_Small JP2
-U 1 1 60EA6557
-P 2850 1850
-F 0 "JP2" H 2850 2035 50  0001 C CNN
-F 1 "MONO+" H 2850 1900 50  0000 C CNN
-F 2 "Connector_PinHeader_2.54mm:PinHeader_1x02_P2.54mm_Vertical" H 2850 1850 50  0001 C CNN
-F 3 "~" H 2850 1850 50  0001 C CNN
-	1    2850 1850
-	0    1    1    0
-$EndComp
-$Comp
-L Device:Jumper_NO_Small JP1
-U 1 1 60EA7E42
-P 2800 1600
-F 0 "JP1" H 2800 1785 50  0001 C CNN
-F 1 "MONO-" H 2800 1650 50  0000 C CNN
-F 2 "Connector_PinHeader_2.54mm:PinHeader_1x02_P2.54mm_Vertical" H 2800 1600 50  0001 C CNN
-F 3 "~" H 2800 1600 50  0001 C CNN
-	1    2800 1600
-	0    1    1    0
-$EndComp
-Connection ~ 2850 1750
-Wire Wire Line
-	2850 1750 2700 1750
-Connection ~ 2850 1950
-Wire Wire Line
-	2850 1950 2700 1950
-Wire Wire Line
-	3000 1300 3250 1300
-Wire Wire Line
-	2800 1500 2800 1450
-Connection ~ 2800 1450
-Wire Wire Line
-	2800 1450 2700 1450
-Wire Wire Line
-	2800 1700 2800 1850
-Connection ~ 2800 1850
-Wire Wire Line
-	2800 1850 2700 1850
-Wire Wire Line
-	3850 1150 4450 1150
-Wire Wire Line
-	4450 1150 4450 2000
-Wire Wire Line
 	4450 2000 4900 2000
 Wire Wire Line
-	3850 1300 4500 1300
-Wire Wire Line
-	4500 1300 4500 1900
-Wire Wire Line
 	4500 1900 4900 1900
 Wire Wire Line
-	3850 1950 4550 1950
+	3850 1950 3900 1950
 Wire Wire Line
 	4550 1950 4550 1200
@@
 	4550 1200 4900 1200
 Wire Wire Line
-	3850 1800 4600 1800
+	3850 1800 4300 1800
 Wire Wire Line
 	4600 1800 4600 1300
@@
 	4900 1800 4850 1800
 Wire Wire Line
-	4850 1800 4850 1450
+	4850 1800 4850 1550
 Wire Wire Line
 	4850 1450 4900 1450
@@
 Wire Wire Line
 	4900 1450 4900 1500
+Wire Wire Line
+	5200 2200 4350 2200
+Wire Wire Line
+	4350 2200 4350 2150
+Wire Wire Line
+	4350 2150 3850 2150
+Wire Wire Line
+	4100 1550 4850 1550
+Connection ~ 4100 1550
+Connection ~ 4850 1550
+Wire Wire Line
+	4850 1550 4850 1450
+Wire Wire Line
+	2700 1750 2950 1750
+Wire Wire Line
+	2700 1950 3100 1950
+Wire Wire Line
+	2700 1850 3050 1850
+Wire Wire Line
+	2700 1450 3000 1450
+Wire Wire Line
+	3350 1000 3350 1150
+Wire Wire Line
+	2950 1150 3350 1150
+Wire Wire Line
+	4050 1000 3400 1000
+Wire Wire Line
+	3400 1000 3400 1300
+Wire Wire Line
+	3000 1300 3400 1300
+Wire Wire Line
+	4450 1100 3100 1100
+Wire Wire Line
+	3100 1100 3100 850
+Wire Wire Line
+	4450 1100 4450 2000
+Wire Wire Line
+	4500 1050 3800 1050
+Wire Wire Line
+	3800 1050 3800 850
+Wire Wire Line
+	4500 1050 4500 1900
+Wire Wire Line
+	3600 850  3600 1250
+Wire Wire Line
+	3600 1250 3900 1250
+Wire Wire Line
+	3900 1250 3900 1950
+Connection ~ 3900 1950
+Wire Wire Line
+	3900 1950 4550 1950
+Wire Wire Line
+	4300 850  4300 1800
+Connection ~ 4300 1800
+Wire Wire Line
+	4300 1800 4600 1800
 $EndSCHEMATC
